File: electrical/autopilot.kicad_sch (KiCad schematic)
At the start: 5 parts

Commit message: Simplified lighting ground
Changed lines of the file:
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@@
-    (stroke (width 0) (type default))
-  )
-  (wire (pts (xy 204.47 29.21) (xy 196.85 29.21))
     (stroke (width 0) (type default))
   )
@@
     (stroke (width 0) (type default))
   )
+  (wire (pts (xy 196.85 29.21) (xy 204.47 29.21))
+    (stroke (width 0) (type default))
+  )
