File: electrical/autopilot.kicad_sch (KiCad schematic)
At the start: 5 parts

Commit message: Changed grounds and canbuses to be in/out when applicable.
Other:
- note added: "Canbus Termination"
Changed lines of the file:
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@@
     (stroke (width 0) (type default))
+  )
+  (text "Canbus Termination" (at 67.31 160.02 0)
+    (effects (font (size 1.27 1.27)) (justify left bottom))
   )
   (global_label "GND" (shape passive) (at 88.9 148.59 0) (fields_autoplaced)
@@
     )
   )
-  (hierarchical_label "CAN_HI_IN" (shape passive) (at 172.72 33.02 180) (fields_autoplaced)
+  (hierarchical_label "CAN_HI_IN" (shape input) (at 172.72 33.02 180) (fields_autoplaced)
     (effects (font (size 1.27 1.27)) (justify right))
   )
@@
     (effects (font (size 1.27 1.27)) (justify left))
   )
-  (hierarchical_label "CAN_LO_IN" (shape passive) (at 172.72 35.56 180) (fields_autoplaced)
+  (hierarchical_label "CAN_LO_IN" (shape input) (at 172.72 35.56 180) (fields_autoplaced)
     (effects (font (size 1.27 1.27)) (justify right))
   )
@@
     (effects (font (size 1.27 1.27)) (justify left))
   )
-  (hierarchical_label "TOGA_IN" (shape passive) (at 196.85 44.45 180) (fields_autoplaced)
+  (hierarchical_label "TOGA_IN" (shape input) (at 196.85 44.45 180) (fields_autoplaced)
     (effects (font (size 1.27 1.27)) (justify right))
   )
@@
     (effects (font (size 1.27 1.27)) (justify left))
   )
-  (hierarchical_label "GND_BUS" (shape passive) (at 30.48 200.66 180) (fields_autoplaced)
+  (hierarchical_label "GND_BUS" (shape input) (at 30.48 200.66 180) (fields_autoplaced)
     (effects (font (size 1.27 1.27)) (justify right))
   )

Commit message: Removed GAD 27 and just use VP-X. Not worth it for lights control and better wig-wag. VP-X is good enough and frees up breakers.
Connections:
- net LIGHTING_HI: no longer names the net of GMC507.P7001_11 (LIGHTING_BUS_HI)
Changed lines of the file:
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@@
   (title_block
     (title "Autopilot")
-    (date "2024-02-08")
-    (rev "0.9")
+    (date "2024-02-13")
+    (rev "0.91")
     (company "N915SN Angry Bird")
   )
@@
     (stroke (width 0) (type default))
   )
-  (wire (pts (xy 204.47 46.99) (xy 196.85 46.99))
-    (stroke (width 0) (type default))
-  )
   (wire (pts (xy 204.47 35.56) (xy 179.07 35.56))
     (stroke (width 0) (type default))
@@
     (effects (font (size 1.27 1.27)) (justify right))
   )
-  (hierarchical_label "LIGHTING_HI" (shape input) (at 196.85 46.99 180) (fields_autoplaced)
-    (effects (font (size 1.27 1.27)) (justify right))
-  )
