File: electrical/multifunction.kicad_sch (KiCad schematic)
At the start: 16 parts

Commit message: Simplified lighting ground
Connections:
- net LIGHTING_GND: no longer names the net of CABIN_CTL.3, GAD27.P271_38 (LIGHTING_BUS_GROUND), PANEL_CTL.3
Changed lines of the file:
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@@
   (junction (at 96.52 35.56) (diameter 0) (color 0 0 0 0)
-  )
-  (junction (at 92.71 129.54) (diameter 0) (color 0 0 0 0)
   )
   (no_connect (at 81.28 38.1))
@@
     (stroke (width 0) (type default))
   )
-  (wire (pts (xy 95.25 130.81) (xy 92.71 130.81))
-    (stroke (width 0) (type default))
-  )
   (wire (pts (xy 81.28 147.32) (xy 95.25 147.32))
     (stroke (width 0) (type default))
@@
     (stroke (width 0) (type default))
   )
-  (wire (pts (xy 92.71 129.54) (xy 120.65 129.54))
+  (wire (pts (xy 81.28 129.54) (xy 120.65 129.54))
     (stroke (width 0) (type default))
   )
@@
     (stroke (width 0) (type default))
   )
-  (wire (pts (xy 81.28 129.54) (xy 92.71 129.54))
-    (stroke (width 0) (type default))
-  )
   (wire (pts (xy 88.9 203.2) (xy 88.9 161.29))
     (stroke (width 0) (type default))
@@
   )
   (wire (pts (xy 160.02 128.27) (xy 160.02 123.19))
-    (stroke (width 0) (type default))
-  )
-  (wire (pts (xy 92.71 130.81) (xy 92.71 129.54))
     (stroke (width 0) (type default))
   )
@@
     (effects (font (size 1.27 1.27)) (justify left))
   )
-  (hierarchical_label "LIGHTING_GND" (shape passive) (at 95.25 130.81 0) (fields_autoplaced)
-    (effects (font (size 1.27 1.27)) (justify left))
-  )

Commit message: Updated with overview
Other:
- title: Multifunction Flaps, Lights & Trim -> Flaps, Lights & Trim
Changed lines of the file:
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@@
   (paper "USLetter" portrait)
   (title_block
-    (title "Multifunction Flaps, Lights & Trim")
+    (title "Flaps, Lights & Trim")
     (date "2024-02-03")
     (rev "0.5")
