File: electrical/multifunction.kicad_sch (KiCad schematic)
At the start: 16 parts

Commit message: Made minimal, and removed everything not needed. want to add GMC 507 back.
Parts:
- removed LANDING1_LT, LANDING2_LT: ~, symbol flyerx:Bulb
- removed PITCH_TRIM, SLATS: Motor_DC, symbol Motor:Motor_DC
- removed PITCH_TRIM_DN_SW, PITCH_TRIM_UP_SW, SLATS_IN_SW, SLATS_OUT_SW: SW_Push, symbol Switch:SW_Push
Connections:
- net GND: no longer GAD27.P272_2 (PITCH_TRIM_POWER_GND), GAD27.TB_6 (FLAP_POWER_GROUND)
- net LANDING_PWR: no longer names the net of GAD27.TB_3 (LIGHT_1_POWER)
- net LANDING_PWR: no longer GAD27.TB_4 (LIGHT_2_POWER)
- net PITCH_TRIM_MOTOR_1_OUT: no longer names the net of GAD27.P272_11 (PITCH_TRIM_OUT_1)
- net PITCH_TRIM_MOTOR_2_OUT: no longer names the net of GAD27.P272_12 (PITCH_TRIM_OUT_2)
- net TOGA_IN: no longer names the net of GAD27.P271_9 (DISCRETE_IN_1)
- net TRIM_FLAPS_PWR: no longer names the net of GAD27.P272_1 (PITCH_TRIM_POWER_IN)
- net TRIM_FLAPS_PWR: no longer GAD27.TB_5 (FLAP_POWER_IN)
Other:
- note removed: "Route through GSA28 Servos"
