File: electrical/navigator.kicad_sch (KiCad schematic)
At the start: 5 parts

Commit message: Changed grounds and canbuses to be in/out when applicable.
Changed lines of the file:
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@@
     (effects (font (size 1.27 1.27)) (justify left))
   )
-  (hierarchical_label "CAN_LO_OUT" (shape bidirectional) (at 129.54 45.72 180) (fields_autoplaced)
+  (hierarchical_label "CAN_LO_OUT" (shape output) (at 129.54 45.72 180) (fields_autoplaced)
     (effects (font (size 1.27 1.27)) (justify right))
   )
-  (hierarchical_label "CAN_HI_OUT" (shape bidirectional) (at 129.54 43.18 180) (fields_autoplaced)
+  (hierarchical_label "CAN_HI_OUT" (shape output) (at 129.54 43.18 180) (fields_autoplaced)
     (effects (font (size 1.27 1.27)) (justify right))
   )
@@
     (effects (font (size 1.27 1.27)) (justify left))
   )
-  (hierarchical_label "CAN_LO_IN" (shape bidirectional) (at 129.54 34.29 180) (fields_autoplaced)
+  (hierarchical_label "CAN_LO_IN" (shape input) (at 129.54 34.29 180) (fields_autoplaced)
     (effects (font (size 1.27 1.27)) (justify right))
   )
@@
     (effects (font (size 1.27 1.27)) (justify left))
   )
-  (hierarchical_label "CAN_HI_IN" (shape bidirectional) (at 129.54 31.75 180) (fields_autoplaced)
+  (hierarchical_label "CAN_HI_IN" (shape input) (at 129.54 31.75 180) (fields_autoplaced)
     (effects (font (size 1.27 1.27)) (justify right))
   )
@@
     (effects (font (size 1.27 1.27)) (justify right))
   )
-  (hierarchical_label "TOGA_OUT" (shape passive) (at 76.2 175.26 0) (fields_autoplaced)
+  (hierarchical_label "TOGA_OUT" (shape output) (at 76.2 175.26 0) (fields_autoplaced)
     (effects (font (size 1.27 1.27)) (justify left))
   )

Commit message: Removed GAD 27 and just use VP-X. Not worth it for lights control and better wig-wag. VP-X is good enough and frees up breakers.
Connections:
- net LIGHTING_HI: no longer names the net of GPS175.P1751_19 (LIGHTING_BUS_HI)
Changed lines of the file:
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@@
   (paper "A" portrait)
   (title_block
-    (date "2024-02-08")
-    (rev "0.9")
+    (date "2024-02-13")
+    (rev "0.91")
   )
   (junction (at 68.58 31.75) (diameter 0) (color 0 0 0 0)
@@
     (stroke (width 0) (type default))
   )
-  (wire (pts (xy 64.77 153.67) (xy 74.93 153.67))
-    (stroke (width 0) (type default))
-  )
   (wire (pts (xy 130.81 53.34) (xy 158.75 53.34))
     (stroke (width 0) (type default))
@@
     (effects (font (size 1.27 1.27)) (justify left))
   )
-  (hierarchical_label "LIGHTING_HI" (shape input) (at 74.93 153.67 0) (fields_autoplaced)
-    (effects (font (size 1.27 1.27)) (justify left))
-  )
